File: IO Expanders.kicad_sch (KiCad schematic)
At the start: 273 parts, among them J103 Conn_02x08_Odd_Even, J46 Conn_02x08_Odd_Even, J47 Conn_02x08_Odd_Even, J48 Conn_02x08_Odd_Even, U11 IO_EXPANDER_TCA9535PWR, U12 IO_EXPANDER_TCA9535PWR, U13 IO_EXPANDER_TCA9535PWR, U23 IO_EXPANDER_TCA9535PWR

Commit message: Rev A0
REV A0 changes, additionally added STEP files for PAM8302, MAX98357, and JST XH 4 connector for UART. Updated KiCad schematic and PCB files, reorganized BOM and pick-and-place files for new revisions, and refreshed CAM data.
Changed lines of the file:
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@@
 		(title "Main Universal Panel Board")
 		(date "2025-08-06")
-		(rev "X4")
+		(rev "A0")
 		(company "CMSC")
 		(comment 1 "NF 2025")
@@
 	(wire
 		(pts
-			(xy 107.95 269.24) (xy 118.11 269.24)
-		)
-		(stroke
-			(width 0)
-			(type default)
-		)
-	)
-	(wire
-		(pts
 			(xy 156.21 293.37) (xy 153.67 293.37)
 		)
@@
 	(wire
 		(pts
-			(xy 483.87 264.16) (xy 473.71 264.16)
-		)
-		(stroke
-			(width 0)
-			(type default)
-		)
-	)
-	(wire
-		(pts
 			(xy 349.25 170.18) (xy 302.26 170.18)
 		)
@@
 	(wire
 		(pts
-			(xy 483.87 137.16) (xy 473.71 137.16)
-		)
-		(stroke
-			(width 0)
-			(type default)
-		)
-	)
-	(wire
-		(pts
 			(xy 334.01 111.76) (xy 334.01 152.4)
 		)
@@
 	(wire
 		(pts
-			(xy 107.95 134.62) (xy 118.11 134.62)
-		)
-		(stroke
-			(width 0)
-			(type default)
-		)
-	)
-	(wire
-		(pts
 			(xy 358.14 101.6) (xy 340.36 101.6)
 		)
@@
 	(wire
 		(pts
-			(xy 107.95 137.16) (xy 118.11 137.16)
-		)
-		(stroke
-			(width 0)
-			(type default)
-		)
-	)
-	(wire
-		(pts
 			(xy 217.17 133.35) (xy 217.17 101.6)
 		)
@@
 	(wire
 		(pts
-			(xy 483.87 266.7) (xy 473.71 266.7)
-		)
-		(stroke
-			(width 0)
-			(type default)
-		)
-	)
-	(wire
-		(pts
 			(xy 200.66 160.02) (xy 203.2 160.02)
 		)
@@
 	(wire
 		(pts
-			(xy 107.95 264.16) (xy 118.11 264.16)
-		)
-		(stroke
-			(width 0)
-			(type default)
-		)
-	)
-	(wire
-		(pts
 			(xy 284.48 201.93) (xy 284.48 147.32)
 		)
@@
 	)
 	(label "VREF_HIGH"
-		(at 473.71 132.08 0)
+		(at 473.71 269.24 0)
 		(effects
 			(font
@@
 	)
 	(label "VREF_HIGH"
-		(at 473.71 269.24 0)
+		(at 473.71 132.08 0)
 		(effects
 			(font
@@
 	)
 	(label "VREF_HIGH"
-		(at 473.71 134.62 0)
+		(at 118.11 266.7 180)
 		(effects
 			(font
 				(size 1.27 1.27)
 			)
-			(justify left bottom)
+			(justify right bottom)
 		)
 	)
 	(label "VREF_HIGH"
-		(at 118.11 266.7 180)
+		(at 292.1 231.14 180)
 		(effects
 			(font
@@
 	)
 	(label "VREF_HIGH"
-		(at 292.1 231.14 180)
+		(at 473.71 134.62 0)
 		(effects
 			(font
 				(size 1.27 1.27)
 			)
-			(justify right bottom)
+			(justify left bottom)
 		)
 	)
@@
 		)
 	)
-	(hierarchical_label "GND"
-		(shape input)
-		(at 483.87 264.16 0)
-		(effects
-			(font
-				(size 1.27 1.27)
-			)
-			(justify left)
-		)
-	)
 	(hierarchical_label "VCC"
 		(shape input)
@@
 	(hierarchical_label "GND"
 		(shape input)
+		(at 473.71 266.7 0)
+		(effects
+			(font
+				(size 1.27 1.27)
+			)
+			(justify left)
+		)
+	)
+	(hierarchical_label "GND"
+		(shape input)
+		(at 118.11 269.24 180)
+		(effects
+			(font
+				(size 1.27 1.27)
+			)
+			(justify right)
+		)
+	)
+	(hierarchical_label "GND"
+		(shape input)
 		(at 233.68 226.06 0)
 		(effects
@@
 		)
 	)
+	(hierarchical_label "GND"
+		(shape input)
+		(at 473.71 264.16 0)
+		(effects
+			(font
+				(size 1.27 1.27)
+			)
+			(justify left)
+		)
+	)
 	(hierarchical_label "VCC"
 		(shape input)
@@
 		)
 	)
+	(hierarchical_label "GND"
+		(shape input)
+		(at 473.71 137.16 0)
+		(effects
+			(font
+				(size 1.27 1.27)
+			)
+			(justify left)
+		)
+	)
 	(hierarchical_label "SDA"
 		(shape input)
@@
 		)
 	)
-	(hierarchical_label "GND"
-		(shape input)
-		(at 483.87 137.16 0)
-		(effects
-			(font
-				(size 1.27 1.27)
-			)
-			(justify left)
-		)
-	)
 	(hierarchical_label "VCC"
 		(shape input)
@@
 		)
 	)
+	(hierarchical_label "GND"
+		(shape input)
+		(at 118.11 264.16 180)
+		(effects
+			(font
+				(size 1.27 1.27)
+			)
+			(justify right)
+		)
+	)
 	(hierarchical_label "VCC"
 		(shape input)
@@
 		)
 	)
-	(hierarchical_label "GND"
-		(shape input)
-		(at 107.95 137.16 180)
-		(effects
-			(font
-				(size 1.27 1.27)
-			)
-			(justify right)
-		)
-	)
 	(hierarchical_label "VCC"
 		(shape input)
@@
 	(hierarchical_label "GND"
 		(shape input)
+		(at 118.11 137.16 180)
+		(effects
+			(font
+				(size 1.27 1.27)
+			)
+			(justify right)
+		)
+	)
+	(hierarchical_label "GND"
+		(shape input)
 		(at 184.15 251.46 0)
 		(effects
@@
 		)
 	)
-	(hierarchical_label "GND"
-		(shape input)
-		(at 107.95 269.24 180)
-		(effects
-			(font
-				(size 1.27 1.27)
-			)
-			(justify right)
-		)
-	)
 	(hierarchical_label "VCC"
 		(shape input)
@@
 	(hierarchical_label "GND"
 		(shape input)
-		(at 241.3 284.48 0)
+		(at 118.11 134.62 180)
 		(effects
 			(font
 				(size 1.27 1.27)
 			)
-			(justify left)
+			(justify right)
 		)
 	)
 	(hierarchical_label "GND"
 		(shape input)
-		(at 425.45 182.88 180)
+		(at 241.3 284.48 0)
 		(effects
 			(font
 				(size 1.27 1.27)
 			)
-			(justify right)
+			(justify left)
 		)
 	)
 	(hierarchical_label "GND"
 		(shape input)
-		(at 367.03 83.82 180)
+		(at 425.45 182.88 180)
 		(effects
 			(font
@@
 	(hierarchical_label "GND"
 		(shape input)
-		(at 483.87 266.7 0)
+		(at 367.03 83.82 180)
 		(effects
 			(font
 				(size 1.27 1.27)
 			)
-			(justify left)
+			(justify right)
 		)
 	)
@@
 	(hierarchical_label "GND"
 		(shape input)
-		(at 107.95 264.16 180)
-		(effects
-			(font
-				(size 1.27 1.27)
-			)
-			(justify right)
-		)
-	)
-	(hierarchical_label "GND"
-		(shape input)
 		(at 241.3 152.4 0)
 		(effects
@@
 		(effects
 			(font
-				(size 1.27 1.27)
-			)
-			(justify right)
-		)
-	)
-	(hierarchical_label "GND"
-		(shape input)
-		(at 107.95 134.62 180)
-		(effects
-			(font
