File: Main Board.kicad_pcb (KiCad board)
At the start: 4 copper layers, 243.2 x 134 mm, 550 parts, among them J10 Conn_02x07_Odd_Even, J102 Speaker Out, J103 Conn_02x08_Odd_Even, J11 Conn_02x07_Odd_Even, J110 SD Holder MEM2061-01-188-00-A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, J12 Conn_02x07_Odd_Even, J13 Conn_01x03_Pin, J14 Conn_01x03_Pin, J15 Conn_01x03_Pin, J16 Conn_01x03_Pin, J17 Conn_01x03_Pin, J18 Conn_01x03_Pin, J19 Conn_01x03_Pin, J2 I2C_MAIN, J20 Conn_01x03_Pin, J21 Conn_01x03_Pin, J22 Conn_01x03_Pin, J23 Conn_01x03_Pin, J24 Conn_01x03_Pin, J25 Conn_01x03_Pin, J26 Conn_01x03_Pin, J27 Conn_01x03_Pin, J28 Conn_01x03_Pin, J29 Conn_01x03_Pin, J3 I2C_A, J30 Conn_01x03_Pin, J31 Conn_01x03_Pin, J32 Conn_01x03_Pin, J33 Conn_01x03_Pin, J34 Conn_01x03_Pin, J35 Conn_01x03_Pin, J36 Conn_01x03_Pin, J37 Conn_01x03_Pin, J38 Conn_01x03_Pin, J39 Conn_01x03_Pin, J4 I2C_B, J40 Conn_01x03_Pin, J41 Conn_01x03_Pin, J42 Conn_01x03_Pin, J43 Conn_01x03_Pin, J44 Conn_01x03_Pin, J45 VCC Select, J46 Conn_02x08_Odd_Even, J47 Conn_02x08_Odd_Even, J48 Conn_02x08_Odd_Even, J49 NEOPIXEL AUX, J5 Conn_02x07_Odd_Even, J6 Conn_02x07_Odd_Even, J7 Conn_02x07_Odd_Even, J8 Conn_02x07_Odd_Even, J85 I2C_C, J86 I2C_D, J87 I2C_E, J88 Neopixel Header, J89 Servo Header B, J9 Conn_02x07_Odd_Even, J90 Servo Header A, J91 Servo Header C, J92 Servo Header D, J93 I2C_F, J94 I2C_G, J95 I2C_H, J96 UART_EXT, J97 Display 1, J98 Display 2, J99 VIN, Q1 BSS138, Q2 NPN transistor, SW1 SW_Push, SW2 SW_Push, U1 ESP32-S3-WROOM-1-N4, U10 Analog_MUX_CD4067BPWR, U11 IO_EXPANDER_TCA9535PWR, U12 IO_EXPANDER_TCA9535PWR, U13 IO_EXPANDER_TCA9535PWR, U19 Shift Register SN74HCS164PWR, U2 Analog_MUX_CD4067BPWR, U21 I2C_MUX_TCA9548APWR, U22 Ethernet Adapter, U23 IO_EXPANDER_TCA9535PWR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

Commit message: Rev A0
REV A0 changes, additionally added STEP files for PAM8302, MAX98357, and JST XH 4 connector for UART. Updated KiCad schematic and PCB files, reorganized BOM and pick-and-place files for new revisions, and refreshed CAM data.
Parts:
- added J50: RESET EN, Connector_PinHeader_2.54mm:PinHeader_1x02_P2.54mm_Vertical, F.Cu at (168.7, 37.7)
- added P50: Conn_01x05_Pin, Connector_PinHeader_2.54mm:PinHeader_1x05_P2.54mm_Vertical, F.Cu at (120.4, 25.5)
- added P51: Conn_01x07, Connector_PinHeader_2.54mm:PinHeader_1x07_P2.54mm_Vertical, F.Cu at (109.3, 56.6)
- added R231: 100K, Resistor_SMD:R_0603_1608Metric, F.Cu at (90.6, 55.0)
- added R255: 0R, Resistor_SMD:R_0603_1608Metric, F.Cu at (112.6, 35.0)
- added R256: 0R, Resistor_SMD:R_0603_1608Metric, F.Cu at (115.5, 35.0)
- added R257: 0R, Resistor_SMD:R_0603_1608Metric, F.Cu at (118.5, 35.0)
- added R258: 10K, Resistor_SMD:R_0603_1608Metric, F.Cu at (115.8, 30.9)
- added R259: 100K, Resistor_SMD:R_0603_1608Metric, F.Cu at (112.2, 30.9)
- added R260: 100K, Resistor_SMD:R_0603_1608Metric, F.Cu at (112.2, 28.1)
- added TP36: TestPoint, Connector_Pin:Pin_D1.0mm_L10.0mm, F.Cu at (167.0, 33.2)
- added TP37: TestPoint, Connector_Pin:Pin_D1.0mm_L10.0mm, F.Cu at (174.1, 33.1)
- moved J96 2.41 mm to (103.0, 29.3)
- moved TP26 0.24 mm to (114.7, 55.0)
Connections:
- net Net-(U1-EN) renamed /MCU_RESET
- net Net-(U1-IO42) renamed /I2S_SD
- J1 pad CTS: /CTS -> /BOOTSEL
- J1 pad RTS: /RTS -> Net-(J50-Pin_2)
- J1 pad RXD: /RXD -> /TXD
- J1 pad TXD: /TXD -> /RXD
- SW1 pad 1: Net-(U1-IO0) -> /BOOTSEL
- TP13 pad 1: unconnected-(TP13-Pad1) -> /I2S_LRCLK
- U1 pad 26: unconnected-(TP13-Pad1) -> /I2S_LRCLK
- U1 pad 27: Net-(U1-IO0) -> /BOOTSEL
- U11 pad 22: /I2C_SCK_MAIN -> /I2C_SCK_A
- U11 pad 23: /I2C_SDA_MAIN -> /I2C_SDA_A
- U12 pad 22: /I2C_SCK_MAIN -> /I2C_SCK_A
- U12 pad 23: /I2C_SDA_MAIN -> /I2C_SDA_A
- U13 pad 22: /I2C_SCK_MAIN -> /I2C_SCK_A
- U13 pad 23: /I2C_SDA_MAIN -> /I2C_SDA_A
- U23 pad 22: /I2C_SCK_MAIN -> /I2C_SCK_A
- U23 pad 23: /I2C_SDA_MAIN -> /I2C_SDA_A
Routing:
- net /I2S_LRCLK: track 0.00 -> 151.1 mm, vias 0 -> 2
- net /I2S_SD: track 18.9 -> 154.6 mm, vias 0 -> 4
- net /Speaker_Out: track 18.6 -> 128.0 mm, vias 0 -> 1
- net /I2C_SCK_A: track 31.7 -> 128.1 mm, vias 0 -> 6
- net /I2C_SDA_A: track 36.2 -> 124.8 mm, vias 0 -> 5
- net /CTS: track 32.7 -> 116.1 mm, vias 1 -> 3
- net /RTS: track 33.2 -> 99.4 mm, vias 1 -> 4
- net /BOOTSEL: track 0.00 -> 62.1 mm, vias 0 -> 2
- net /I2C_SCK_MAIN: track 178.9 -> 117.9 mm
- net /I2C_SDA_MAIN: track 187.9 -> 129.0 mm
- net +5V_SERVO: track 67.6 -> 120.0 mm
- net Net-(J50-Pin_2): track 0.00 -> 51.7 mm
- net Net-(U1-IO0): track 37.3 -> 0.00 mm, vias 1 -> 0
- net +5V_NEOPIXEL: track 276.9 -> 308.4 mm, vias 1 -> 3
- net unconnected-(TP13-Pad1): track 29.1 -> 0.00 mm
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Other:
- board text added: "Main Panel Board NF 1-7-26 REV A0"
- board text added: "PROG RESET EN"
- board text removed: "Main Panel Board NF 8-23-25 REV X4"
